File: SST60.kicad_pcb (KiCad board)
At the start: 2 copper layers, 284.7 x 94.2 mm, 204 parts, among them J1 SM04B, J2 SWD, SW1 Boot, SW2 Reset, U1 RP2040, U2 W25Q128JVS, U3 XC6206PxxxMR, U4 PRTR5V0U2X, U5 74AHCT1G125, Y1 12MHz

Commit message: fixed missing trace
Parts:
- removed D60: D_Small, Diode_SMD:D_SOD-123
- removed the ISO at (284.2, 87.3)
- removed the ISO at (305.6, 77.8)
- moved D38 5.39 mm to (183.1, 127.1)
- moved D78 4.40 mm to (192.0, 123.8)
Routing:
- net col5: track 407.5 -> 294.6 mm
- net col9: track 440.7 -> 345.7 mm
- net col4: track 314.8 -> 238.0 mm
- net +5V: track 742.3 -> 701.5 mm
- net col1: track 102.3 -> 78.5 mm
- net col6: track 351.3 -> 330.4 mm
- net Net-(D64-Pad2): track 19.8 -> 7.41 mm
- net col12: track 325.6 -> 335.0 mm
- net Net-(D76-Pad3): track 39.1 -> 44.1 mm
- net Net-(D33-Pad2): track 3.99 -> 0.00 mm
- net Net-(D60-Pad2): track 3.99 -> 0.00 mm
- net Net-(D6-Pad2): track 3.99 -> 0.00 mm
- net Net-(D38-Pad2): track 18.4 -> 22.2 mm
- net +3V3: track 218.0 -> 214.2 mm
- net GND: track 117.7 -> 114.3 mm, vias 94 -> 93
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